File: KiCad Project Files/SST60.kicad_pcb (KiCad board)
At the start: 2 copper layers, 284.7 x 94.2 mm, 181 parts, among them J1 SM04B, J2 SWD, SW1 Boot, SW2 Reset, U1 RP2040, U2 W25Q128JVS, U3 XC6206PxxxMR, U4 PRTR5V0U2X, U5 74AHCT1G125, Y1 12MHz

Commit message: Error Cleanup
Resolved all errors in sch, and most errors in pcb, except "intentional" ones concerning H1.
Will readdress rule changes and violations once attempting to submit to fab house.
Parts:
- moved USB1 0.35 mm to (50.5, 38.7)
- moved R_Flash1 0.31 mm to (76.9, 65.9)
Routing:
- net GND: track 112.4 -> 111.4 mm
- net VCC: track 15.6 -> 15.1 mm
- net D-: track 41.5 -> 42.0 mm
Other:
- board text added: "Ol' Sweepy was here"
- board text removed: "Old Sweepy was here"

Commit message: Component updates
Updates to components to facilitate JLC PCB process.
Parts:
- C_1V-Decoup2, C_1V-Decoup3, C_3V-Decoup3, C_3V-Decoup4, C_3V-Decoup5, C_3V-Decoup6, C_3V-Decoup7, C_3V-Decoup8, C_3V-Decoup9, C_Flash1: value .1u -> 100n
- D1, D10, D11, D12, D13, D14, D15, D16, D17, D18, D19, D2, D20, D21, D22, D23, D25, D26, D27, D28, D3, D30, D31, D32, D33, D34, D35, D36, D37, D38, D39, D4, D40, D41, D42, D43, D44, D45, D46, D48, D49, D5, D50, D51, D53, D54, D55, D56, D57, D58, D59, D6, D61, D62, D63, D64, D65, D66, D67, D68, D7, D8: value D_Small -> 1N4148
- SW1: value Boot -> TL3342F450QG
- SW2: value Reset -> TL3342F450QG

Commit message: Further Component Updates
More updating of components to decide what is and isn't included in output BOM and Placement files, as well as other component values, to smooth out wrinkles with JLC PCB process.
Parts:
- J1: value SM04B -> SM04B-SRSS-TB(LF)(SN)
Changed lines of the file:
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@@
 		(sheetname "Misc")
 		(sheetfile "Misc.kicad_sch")
-		(attr exclude_from_pos_files)
+		(attr exclude_from_pos_files exclude_from_bom)
 		(fp_line
 			(start -142.342492 -47.624993)
@@
 		(fp_arc
 			(start 40.316512 44.575)
-			(mid 41.488417 42.895045)
+			(mid 41.488415 42.89505)
 			(end 43.432509 42.249999)
 			(stroke
@@
 		(fp_arc
 			(start 43.432509 -47.299996)
-			(mid 41.48841 -47.94505)
+			(mid 41.488431 -47.945059)
 			(end 40.316512 -49.624993)
 			(stroke
@@
 		(fp_arc
 			(start 43.686507 -47.299996)
-			(mid 43.964139 -47.245144)
+			(mid 43.96415 -47.245156)
 			(end 44.199507 -47.088006)
 			(stroke
@@
 		(fp_arc
 			(start 44.189513 42.047)
-			(mid 43.96505 42.196759)
+			(mid 43.96505 42.19677)
 			(end 43.700514 42.249999)
 			(stroke
@@
 		(fp_arc
 			(start 126.825499 42.249999)
-			(mid 126.475888 42.180152)
+			(mid 126.475882 42.180158)
 			(end 126.179503 41.981997)
 			(stroke
@@
 		(fp_arc
 			(start 130.2825 42.249999)
-			(mid 132.226574 42.895067)
+			(mid 132.226596 42.895058)
 			(end 133.398497 44.575)
 			(stroke
@@
 		(solder_paste_margin 0.05)
 		(clearance 0.05)
-		(attr through_hole)
+		(attr through_hole exclude_from_pos_files exclude_from_bom)
 		(fp_line
 			(start -4.47 7.3)
@@
 		(sheetname "Misc")
 		(sheetfile "Misc.kicad_sch")
-		(attr through_hole exclude_from_pos_files)
+		(attr through_hole exclude_from_pos_files exclude_from_bom)
 		(fp_line
 			(start 1.33 -1.27)
@@
 		(sheetname "USB & Power")
 		(sheetfile "USBnPower.kicad_sch")
-		(attr smd)
+		(attr smd exclude_from_pos_files exclude_from_bom)
 		(fp_line
 			(start -0.153641 0.38)
@@
 			)
 		)
-		(property "Value" "SM04B"
+		(property "Value" "SM04B-SRSS-TB(LF)(SN)"
 			(at 0 -3.98 90)
 			(layer "B.Fab")
@@
 		(sheetname "USB & Power")
 		(sheetfile "USBnPower.kicad_sch")
-		(attr smd exclude_from_pos_files)
+		(attr smd)
 		(fp_line
 			(start -3.11 1.785)
@@
 		(sheetname "USB & Power")
 		(sheetfile "USBnPower.kicad_sch")
-		(attr smd)
+		(attr smd exclude_from_pos_files exclude_from_bom)
 		(fp_line
 			(start -0.153641 -0.38)
