File: KiCad Project Files/SST60.kicad_pcb (KiCad board)
At the start: 2 copper layers, 284.7 x 94.2 mm, 181 parts, among them J1 SM04B-SRSS-TB(LF)(SN), J2 SWD, SW1 TL3342F450QG, SW2 TL3342F450QG, U1 RP2040, U2 W25Q128JVS, U3 XC6206PxxxMR, U4 PRTR5V0U2X, U5 74AHCT1G125, Y1 12MHz

Commit message: Shifted JST
This update shifts the JST connected to be placed similar to another reference keyboard, to accommodate a custom milled enclosure - also removes flex cuts -- this is now the default project file design, but older valid production exports are still stored.
Parts:
- moved J1 77.8 mm to (135.9, 60.3)
Routing:
- net col7: track 606.5 -> 212.6 mm
- net col6: track 355.2 -> 175.1 mm
- net col8: track 368.1 -> 210.6 mm
- net col5: track 298.5 -> 156.2 mm
- net col9: track 348.7 -> 228.5 mm
- net col4: track 241.9 -> 136.8 mm
- net col10: track 329.7 -> 247.2 mm
- net +5V: track 735.8 -> 817.8 mm
- net D+: track 40.0 -> 120.7 mm
- net D-: track 42.0 -> 122.2 mm
- net col11: track 366.0 -> 285.8 mm
- net col3: track 182.1 -> 114.6 mm
- net col2: track 156.4 -> 126.5 mm
- net col12: track 316.5 -> 308.1 mm
